Commit message: Fixed mesh file and transform.

File: op3_description/urdf/robotis_op3.d435.visuals.xacro (robot description, xacro)
@@ -206,5 +206,5 @@
   <!-- head tilt joint -->
   <xacro:macro name="insert_mesh_head_tilt_link">
-    <origin xyz="0 -0.019 0" rpy="${-pi*0.5} 0 0" />
+    <origin xyz="0 0 0" rpy="0 0 0" />
     <geometry>
       <mesh filename="package://op3_description/meshes/h2_d435.dae"  scale="1.000 1.000 1.000"/>
