Commit message: Added camera_base_joint, link and mesh.

File: op3_description/urdf/robotis_op3.d435.structure.head.xacro (robot description, xacro)
@@ -59,9 +59,26 @@
   <link name="cam_gazebo_link">
   </link>
-  <xacro:include filename="$(find realsense2_camera)/urdf/_d435.urdf.xacro"/>
-  <sensor_d435 parent="head_tilt_link">
-    <!-- <origin xyz="0.018 0 0.05275" rpy="${pi*0.5} ${-pi*0.5} 0"/> -->
-    <origin xyz="-0.0041 -0.019 0.04025" rpy="0 0 0"/>
-  </sensor_d435>
+  <!-- camera base joint -->
+  <joint name="camera_base" type="fixed">
+    <parent link="head_tile_link"/>
+    <child link="camera_base_link"/>
+    <origin xyz="0 0 0" rpy="0 0 0" /> <!-- need to be modified -->
+  </joint>
+  <!-- camera base link -->
+  <link name="camera_base_link">
+    <visual>
+      <xacro:insert_mesh_camera_base_link />
+    </visual>
+    <collision>
+      <xacro:insert_mesh_camera_base_link />
+    </collision>
+    <!-- <inertial> -->
+    <!--   <xacro:insert_inertia_camera_base_link /> -->
+    <!-- </inertial> -->
+  </link>
+  <!-- <xacro:include filename="$(find realsense2_camera)/urdf/_d435.urdf.xacro"/> -->
+  <!-- <sensor_d435 parent="head_tilt_link"> -->
+  <!--   <origin xyz="-0.0041 -0.019 0.04025" rpy="0 0 0"/> -->
+  <!-- </sensor_d435> -->
   </xacro:macro>
 </robot>

File: op3_description/urdf/robotis_op3.d435.visuals.xacro (robot description, xacro)
@@ -214,3 +214,13 @@
     <!-- </material> -->
   </xacro:macro>
+  <!-- camera base joint -->
+  <xacro:macro name="insert_mesh_camera_base_link">
+    <origin xyz="0 0 0" rpy="0 0 0" />
+    <geometry>
+      <mesh filename="package://realsense2_camera//meshes/d435.dae"  scale="1.000 1.000 1.000"/>
+    </geometry>
+    <!-- <material name="Grey"> -->
+    <!--   <color rgba="0.60 0.60 0.60 1.0"/> -->
+    <!-- </material> -->
+  </xacro:macro>
 </robot>

Commit message: fixed typo.

File: op3_description/urdf/robotis_op3.d435.structure.head.xacro (robot description, xacro)
@@ -61,5 +61,5 @@
   <!-- camera base joint -->
   <joint name="camera_base" type="fixed">
-    <parent link="head_tile_link"/>
+    <parent link="head_tilt_link"/>
     <child link="camera_base_link"/>
     <origin xyz="0 0 0" rpy="0 0 0" /> <!-- need to be modified -->

Commit message: Modified launch file.

File: op3_description/urdf/robotis_op3.d435.structure.head.xacro (robot description, xacro)
@@ -63,5 +63,5 @@
     <parent link="head_tilt_link"/>
     <child link="camera_base_link"/>
-    <origin xyz="0 0 0" rpy="0 0 0" /> <!-- need to be modified -->
+    <origin xyz="${-0.0041+0.0149} -0.019 ${0.04025+0.0125}" rpy="0 0 0"/>
   </joint>
   <!-- camera base link -->

File: op3_description/urdf/robotis_op3.d435.visuals.xacro (robot description, xacro)
@@ -216,5 +216,5 @@
   <!-- camera base joint -->
   <xacro:macro name="insert_mesh_camera_base_link">
-    <origin xyz="0 0 0" rpy="0 0 0" />
+    <origin xyz="0 0 0" rpy="${pi/2} 0 ${pi/2}" />
     <geometry>
       <mesh filename="package://realsense2_camera//meshes/d435.dae"  scale="1.000 1.000 1.000"/>
