Commit message: Added model files.

File: op3_description/urdf/robotis_op3.d435.ft.structure.lleg.xacro (robot description, xacro)
@@ -142,10 +142,10 @@
     <parent link="l_ank_roll_link"/>
     <child link="l_ank_ft_link"/>
-    <origin xyz="0.0241 0 -0.025" rpy="${pi} ${pi} ${-pi/2}" />
+    <origin xyz="0.022 0 -0.028" rpy="${pi} ${pi} ${pi}" />
     <!-- <axis xyz="0 0 1" /> -->
     <!-- <limit effort="1000" velocity="100" lower="${-pi*0.9}" upper="${pi*0.9}" /> -->
     <!-- <dynamics damping="0.1" friction="0.0" /> -->
   </joint>
-  <xacro:insert_transmission name="l_ank_roll" />
+  <!-- <xacro:insert_transmission name="l_ank_roll" /> -->
   <link name="l_ank_ft_link"/>
   </xacro:macro>

File: op3_description/urdf/robotis_op3.d435.ft.structure.rleg.xacro (robot description, xacro)
@@ -142,10 +142,10 @@
     <parent link="r_ank_roll_link"/>
     <child link="r_ank_ft_link"/>
-    <origin xyz="0.0241 0 -0.025" rpy="${pi} ${pi} ${pi/2}" />
+    <origin xyz="0.022 0 -0.028" rpy="${pi} ${pi} ${pi}" />
     <!-- <axis xyz="0 0 1" /> -->
     <!-- <limit effort="1000" velocity="100" lower="${-pi*0.9}" upper="${pi*0.9}" /> -->
     <!-- <dynamics damping="0.1" friction="0.0" /> -->
   </joint>
-  <xacro:insert_transmission name="r_ank_roll" />
+  <!-- <xacro:insert_transmission name="r_ank_roll" /> -->
   <link name="r_ank_ft_link"/>
   </xacro:macro>

File: op3_description/urdf/robotis_op3.d435.visuals.xacro (robot description, xacro)
@@ -68,5 +68,5 @@
     <origin xyz="0 0 0" rpy="0 0 0" />
     <geometry>
-      <mesh filename="package://op3_description/meshes/rl6.stl"  scale="0.001 0.001 0.001"/>
+      <mesh filename="package://op3_description/meshes/rl6_ft.stl"  scale="0.001 0.001 0.001"/>
     </geometry>
     <material name="Grey">
@@ -128,5 +128,5 @@
     <origin xyz="0 0 0" rpy="0 0 0" />
     <geometry>
-      <mesh filename="package://op3_description/meshes/ll6.stl"  scale="0.001 0.001 0.001"/>
+      <mesh filename="package://op3_description/meshes/ll6_ft.stl"  scale="0.001 0.001 0.001"/>
     </geometry>
     <material name="Grey">
